File: pcb/rev.A/dendy.kicad_pcb (KiCad board)
At the start: 2 copper layers, 91 x 187 mm, 125 parts, among them J10 FC 60 pin cartridge slot, J2 DB15_Male, J3 RCJ-014, J4 RCJ-014, J5 PJ-322, J6 DB15_Male, J7 DS-210, J8 Conn_01x02, Q1 BC549B, Q2 BC549B, Q3 BC549B, Q4 BC549B, Q5 2N5401, SW1 SW_SPDT, SW2 Button THT, U1 74LS139, U10 MC1458P, U2 74LS373, U3 62256, U4 62256, U5 RP2A03, U6 RP2C02, U7 74LS368, U8 74LS368, U9 LM2596T-ADJ, Y1 21.47727MHz, Y2 26.601712MHz

Commit message: wip pcb rev.A
Parts:
- removed J5: PJ-322, my:PJ-322
- removed JP3: Jumper_2_Open, Connector_PinHeader_2.54mm:PinHeader_1x02_P2.54mm_Vertical
- added C36: 100u, PCM_Capacitor_THT_AKL:CP_Radial_D6.3mm_P2.50mm, F.Cu at (251.4, 200.6)
- added C37: 100n, PCM_Capacitor_THT_AKL:C_Disc_D5.0mm_W2.5mm_P2.50mm, F.Cu at (244.3, 177.8)
- added J1: RCJ-014, my:CUI_RCJ-01X, F.Cu at (182.1, 57.7)
- added L4: 220u/0.2A, PCM_Inductor_THT_AKL:L_Radial_D8.7mm_P5.00mm_Fastron_07HCP, F.Cu at (243.2, 204.3)
- added R44: 47k, PCM_Resistor_THT_AKL:R_Axial_DIN0207_L6.3mm_D2.5mm_P7.62mm_Horizontal, F.Cu at (204.2, 65.4)
- added R45: 10k, PCM_Resistor_THT_AKL:R_Axial_DIN0207_L6.3mm_D2.5mm_P7.62mm_Horizontal, F.Cu at (235.0, 94.0)
- C1, C10, C12, C13, C14, C15, C17, C18, C19, C20, C21, C26, C28, C29, C3, C30, C31, C32, C33, C34, C35, C7, C8, C9: footprint Capacitor_THT_AKL:C_Disc_D5.0mm_W2.5mm_P2.50mm -> PCM_Capacitor_THT_AKL:C_Disc_D5.0mm_W2.5mm_P2.50mm
- C11, C6: footprint Capacitor_THT_AKL:C_Trimmer_GKU_L5.6mm_W5.0mm_P5.8mm -> PCM_Capacitor_THT_AKL:C_Trimmer_GKU_L5.6mm_W5.0mm_P5.8mm
- C16: value 220u -> 100u; footprint Capacitor_THT_AKL:CP_Radial_D6.3mm_P2.50mm -> PCM_Capacitor_THT_AKL:CP_Radial_D6.3mm_P2.50mm
- C2: footprint Capacitor_THT_AKL:CP_Radial_D10.0mm_P5.00mm -> PCM_Capacitor_THT_AKL:CP_Radial_D10.0mm_P5.00mm
- C22, C23, C24, C25, C27, C5: footprint Capacitor_THT_AKL:CP_Radial_D4.0mm_P2.00mm -> PCM_Capacitor_THT_AKL:CP_Radial_D4.0mm_P2.00mm
- C4: footprint Capacitor_THT_AKL:CP_Radial_D8.0mm_P3.50mm -> PCM_Capacitor_THT_AKL:CP_Radial_D8.0mm_P3.50mm
- D2: footprint Diode_THT_AKL:D_DO-41_SOD81_P10.16mm_Horizontal -> PCM_Diode_THT_AKL:D_DO-41_SOD81_P10.16mm_Horizontal
- D3: footprint Diode_THT_AKL:D_DO-201AD_P15.24mm_Horizontal -> PCM_Diode_THT_AKL:D_DO-201AD_P15.24mm_Horizontal
- F1: value 0.5A -> 1A
- L1: footprint Inductor_SMD_AKL:L_12x12mm_H8mm -> PCM_Inductor_SMD_AKL:L_12x12mm_H8mm
- L2, L3: footprint Inductor_THT_AKL:L_Radial_D8.7mm_P5.00mm_Fastron_07HCP -> PCM_Inductor_THT_AKL:L_Radial_D8.7mm_P5.00mm_Fastron_07HCP
- Q1, Q2, Q3, Q4: footprint Package_TO_SOT_THT_AKL:TO-92_Inline_Wide_CBE -> PCM_Package_TO_SOT_THT_AKL:TO-92_Inline_Wide_CBE
- Q5: footprint Package_TO_SOT_THT_AKL:TO-92_Inline_Wide_EBC -> PCM_Package_TO_SOT_THT_AKL:TO-92_Inline_Wide_EBC
- R1: value 100 -> 47k; footprint Resistor_THT_AKL:R_Axial_DIN0207_L6.3mm_D2.5mm_P7.62mm_Horizontal -> PCM_Resistor_THT_AKL:R_Axial_DIN0207_L6.3mm_D2.5mm_P7.62mm_Horizontal
- R10, R11, R12, R13, R14, R15, R16, R17, R18, R19, R2, R20, R21, R22, R23, R24, R25, R26, R27, R28, R29, R3, R30, R31, R32, R33, R34, R35, R36, R37, R38, R39, R4, R40, R41, R42, R43, R5, R6, R7, R8, R9: footprint Resistor_THT_AKL:R_Axial_DIN0207_L6.3mm_D2.5mm_P7.62mm_Horizontal -> PCM_Resistor_THT_AKL:R_Axial_DIN0207_L6.3mm_D2.5mm_P7.62mm_Horizontal
- RN2, RN3: value R_Network05 -> 10k; footprint Resistor_THT_AKL:R_Array_SIP6 -> PCM_Resistor_THT_AKL:R_Array_SIP6
- U1, U7, U8: footprint Package_DIP_AKL:DIP-16_W7.62mm -> PCM_Package_DIP_AKL:DIP-16_W7.62mm
- U10: footprint Package_DIP_AKL:DIP-8_W7.62mm_LongPads -> PCM_Package_DIP_AKL:DIP-8_W7.62mm_LongPads
- U2: footprint Package_DIP_AKL:DIP-20_W7.62mm -> PCM_Package_DIP_AKL:DIP-20_W7.62mm
- U3, U4: footprint Package_DIP_AKL:DIP-28_W7.62mm -> PCM_Package_DIP_AKL:DIP-28_W7.62mm
- U5, U6: footprint Package_DIP_AKL:DIP-40_W15.24mm_Socket -> PCM_Package_DIP_AKL:DIP-40_W15.24mm_Socket
- Y1, Y2: footprint Crystal_AKL:Crystal_HC49-U_Vertical -> PCM_Crystal_AKL:Crystal_HC49-U_Vertical
- moved C17 87.5 mm to (205.8, 75.5), turned to -90 degrees
- moved C16 79.0 mm to (205.8, 87.2)
- moved L3 68.8 mm to (209.5, 95.2), turned to 180 degrees
- moved R4 66.0 mm to (173.2, 143.4)
- moved D5 60.5 mm to (173.2, 146.2)
- moved C5 58.4 mm to (175.6, 204.0), turned to 180 degrees
- moved R24 55.3 mm to (193.3, 70.0), turned to 180 degrees
- moved R43 55.1 mm to (229.3, 103.2), turned to 0 degrees
- moved C10 52.1 mm to (199.8, 216.3)
- moved R40 51.7 mm to (208.4, 190.9), turned to 90 degrees
- moved C33 50.9 mm to (212.8, 110.8)
- moved R32 50.6 mm to (193.3, 83.7), turned to 180 degrees
- moved R17 48.9 mm to (191.9, 80.6), turned to 90 degrees
- moved C26 47.8 mm to (185.0, 75.7), turned to 90 degrees
- moved C27 46.6 mm to (185.0, 78.6), turned to -90 degrees
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Connections:
- C16 pad 1: +5VA -> +5VA_1
- C17 pad 2: +5VA -> +5VA_1
- D5 pad 2: Net-(D5-Pad2) -> Net-(D5-A)
- F1 pad 2: Net-(F1-Pad2) -> Net-(D1-Pad2)
- J4 pad 1: /COMPOSITE -> /SND_R
- J7 pad 2: Net-(D1-Pad2) -> Net-(D1-Pad4)
- J7 pad 3: Net-(D1-Pad2) -> Net-(D1-Pad4)
- L3 pad 2: +5VA -> +5VA_1
- Q4 pad 1: +5VA -> +5VA_2
- R1 pad 1: Net-(JP3-Pad1) -> /SND_R
- R1 pad 2: Net-(C24-Pad1) -> GND
- R14 pad 1: +5VA -> +5VA_2
- R17 pad 1: +5VA -> +5VA_1
- R19 pad 1: +5VA -> +5VA_1
- R27 pad 1: +5VA -> +5VA_1
- R4 pad 2: Net-(D5-Pad2) -> Net-(D5-A)
- SW1 pad 2: Net-(F1-Pad2) -> Net-(SW1-B)
- SW1 pad 3: Net-(D1-Pad4) -> GND
- U1 pad 1: Net-(U1-Pad1) -> GND
- U1 pad 11: Net-(U1-Pad1) -> /~{PPUSEL}
- U1 pad 12: unconnected-(U1-Pad12) -> Net-(D5-A)
- U1 pad 13: /A15 -> /A14
- U1 pad 14: /M2 -> /A13
- U1 pad 15: GND -> Net-(U1A-O1)
- U1 pad 2: /A13 -> /M2
- U1 pad 3: /A14 -> /A15
- U1 pad 4: Net-(D5-Pad2) -> unconnected-(U1A-O0-Pad4)
- U1 pad 5: /~{PPUSEL} -> Net-(U1A-O1)
- U1 pad 7: unconnected-(U1-Pad7) -> /~{ROMSEL}
- U1 pad 9: /~{ROMSEL} -> unconnected-(U1B-O3-Pad9)
- U10 pad 8: +5VA -> +5VA_1
- U3 pad 10: /A7 -> /A0
- U3 pad 11: /D0 -> /D6
- U3 pad 12: /D1 -> /D4
- U3 pad 15: /D7 -> /D0
- U3 pad 16: /D6 -> /D1
- U3 pad 17: /D5 -> /D3
- U3 pad 18: /D4 -> /D5
- U3 pad 19: /D3 -> /D7
- U3 pad 21: /A10 -> /A3
- U3 pad 24: /A9 -> /A8
- U3 pad 25: /A8 -> /A10
- U3 pad 3: /A0 -> /A9
- U3 pad 4: /A1 -> /A7
- U3 pad 5: /A2 -> /A6
- U3 pad 6: /A3 -> /A5
- U3 pad 8: /A5 -> /A2
- U3 pad 9: /A6 -> /A1
- U4 pad 10: /PA7 -> /PA0
- U4 pad 15: /PAD7 -> /PAD3
- U4 pad 16: /PAD6 -> /PAD4
- U4 pad 18: /PAD4 -> /PAD6
- U4 pad 19: /PAD3 -> /PAD7
- U4 pad 21: /VA10 -> /PA4
- U4 pad 24: /PA9 -> /PA7
- U4 pad 25: /PA8 -> /VA10
- U4 pad 3: /PA4 -> /PA6
- U4 pad 4: /PA0 -> /PA5
- U4 pad 5: /PA1 -> /PA8
- U4 pad 6: /PA5 -> /PA9
- U4 pad 7: /PA6 -> /PA3
- U4 pad 9: /PA3 -> /PA1
- U9 pad 5: GND -> Net-(SW1-B)
Routing:
- net Net-(SW1-B): track 0.00 -> 275.6 mm, vias 0 -> 2
- net /~{RESET}: track 0.00 -> 214.0 mm, vias 0 -> 2
- net /COMPOSITE: track 0.00 -> 194.1 mm
- net +5V: track 0.00 -> 158.6 mm
- net /~{IRQ}: track 0.00 -> 120.3 mm
- net /OUT0: track 0.00 -> 108.5 mm, vias 0 -> 1
- net /OUT1: track 0.00 -> 105.7 mm, vias 0 -> 1
- net /M2: track 0.00 -> 103.5 mm, vias 0 -> 1
- net /OUT2: track 0.00 -> 99.7 mm, vias 0 -> 1
- net /R/~{W}: track 0.00 -> 95.4 mm
- net /A10: track 0.00 -> 92.4 mm, vias 0 -> 1
- net /PA7: track 0.00 -> 90.7 mm
- net /PAD7: track 0.00 -> 88.4 mm
- net /PAD5: track 0.00 -> 85.7 mm, vias 0 -> 1
- net /~{JOY2}: track 0.00 -> 84.9 mm
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- added copper zone on B.Cu, net GND
- added copper zone on F.Cu, net GND

Commit message: wip pcb rev.A
Parts:
- removed J8: Conn_01x02, Connector_Molex:Molex_KK-254_AE-6410-02A_1x02_P2.54mm_Vertical
- removed R38, R39, R40, R42: 10k, PCM_Resistor_THT_AKL:R_Axial_DIN0207_L6.3mm_D2.5mm_P7.62mm_Horizontal
- removed RN3: 10k, PCM_Resistor_THT_AKL:R_Array_SIP6
- added C38: 100u, PCM_Capacitor_THT_AKL:CP_Radial_D6.3mm_P2.50mm, F.Cu at (146.6, 183.4)
- added C39: 100u, PCM_Capacitor_THT_AKL:CP_Radial_D6.3mm_P2.50mm, F.Cu at (69.1, 183.4)
- added C40: 100u, PCM_Capacitor_THT_AKL:CP_Radial_D6.3mm_P2.50mm, F.Cu at (131.4, 134.5)
- added C41: 100u, PCM_Capacitor_THT_AKL:CP_Radial_D6.3mm_P2.50mm, F.Cu at (105.4, 134.5)
- added D4: LED, LED_THT:LED_D5.0mm, F.Cu at (105.3, 220.3)
- added RN1: 10k, Resistor_THT:R_Array_SIP9, F.Cu at (81.4, 214.4)
- L2: value 68uH/2A -> 47uH/2A
- RN2: footprint PCM_Resistor_THT_AKL:R_Array_SIP6 -> Resistor_THT:R_Array_SIP9
- moved C36 115.4 mm to (136.8, 186.8), turned to 0 degrees
- moved R6 112.6 mm to (66.4, 188.6), turned to 0 degrees
- moved U8 109.5 mm to (131.8, 204.2)
- moved C29 109.5 mm to (129.4, 201.5)
- moved R41 106.7 mm to (104.1, 139.4), turned to -90 degrees
- moved D1 105.6 mm to (142.0, 64.1)
- moved C18 105.4 mm to (79.0, 149.9), turned to -90 degrees
- moved R18 105.1 mm to (80.0, 76.8)
- moved R21 105.1 mm to (71.0, 76.8)
- moved R22 105.1 mm to (89.0, 76.8)
- moved R26 105.1 mm to (83.0, 76.8)
- moved R29 105.1 mm to (74.0, 76.8)
- moved R30 105.1 mm to (92.0, 76.8)
- moved R34 105.1 mm to (86.0, 84.4)
- moved R35 105.1 mm to (77.0, 84.4)
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Connections:
- J6 pad 4: Net-(RN2-R1) -> Net-(RN2-R5)
- J6 pad 5: Net-(RN3-R5) -> Net-(RN2-R4)
- J6 pad 6: Net-(RN2-R2) -> Net-(RN2-R3)
- J6 pad 7: Net-(RN3-R4) -> Net-(RN2-R2)
- J6 pad 8: Net-(RN2-R3) -> Net-(RN2-R1)
- RN2 pad 5: Net-(J6-P13) -> Net-(RN2-R4)
- RN2 pad 6: unconnected-(RN2-R5-Pad6) -> Net-(RN2-R5)
- U3 pad 11: /D6 -> /D4
- U3 pad 12: /D4 -> /D2
- U3 pad 13: /D2 -> /D0
- U3 pad 15: /D0 -> /D1
- U3 pad 16: /D1 -> /D3
- U3 pad 17: /D3 -> /D5
- U3 pad 18: /D5 -> /D6
- U4 pad 11: /PAD0 -> /PAD7
- U4 pad 12: /PAD1 -> /PAD6
- U4 pad 13: /PAD2 -> /PAD5
- U4 pad 15: /PAD3 -> /PAD4
- U4 pad 16: /PAD4 -> /PAD3
- U4 pad 17: /PAD5 -> /PAD2
- U4 pad 18: /PAD6 -> /PAD1
- U4 pad 19: /PAD7 -> /PAD0
- U4 pad 24: /PA7 -> /PA8
- U4 pad 25: /VA10 -> /PA6
- U4 pad 3: /PA6 -> /VA10
- U4 pad 4: /PA5 -> /PA7
- U4 pad 5: /PA8 -> /PA5
- U8 pad 10: Net-(RN2-R1) -> Net-(RN2-R5)
- U8 pad 12: Net-(RN2-R2) -> Net-(RN2-R3)
- U8 pad 14: Net-(RN2-R3) -> Net-(RN2-R1)
- U8 pad 4: Net-(RN3-R4) -> Net-(RN2-R2)
- U8 pad 6: Net-(RN3-R5) -> Net-(RN2-R4)
Routing:
- net +5V: track 158.6 -> 810.8 mm, vias 0 -> 3
- net /SND_I: track 0.00 -> 201.8 mm, vias 0 -> 2
- net /D4: track 48.5 -> 218.1 mm, vias 0 -> 3
- net /D3: track 56.6 -> 223.4 mm, vias 0 -> 3
- net /D0: track 53.2 -> 208.1 mm, vias 0 -> 3
- net /D1: track 53.6 -> 206.9 mm, vias 0 -> 3
- net /D2: track 47.9 -> 193.1 mm, vias 0 -> 1
- net /PA13: track 0.00 -> 131.9 mm, vias 0 -> 3
- net /M2: track 103.5 -> 234.4 mm, vias 1 -> 5
- net /NPA13: track 0.00 -> 130.0 mm, vias 0 -> 4
- net Net-(J2-P9): track 0.00 -> 88.7 mm
- net /D7: track 59.4 -> 138.9 mm, vias 0 -> 1
- net /D6: track 51.3 -> 130.1 mm, vias 0 -> 1
- net /~{PWR}: track 19.7 -> 90.0 mm
- net /D5: track 57.6 -> 126.9 mm, vias 0 -> 1
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- added copper zone on F.Cu, net +5V
Other:
- outline, holes or cut-outs redrawn
- board text added: "Min clearance: 0.25mm Min track: 0.25mm Min hole: 0.4mm Min annular ring: 0.2mm"
- board text removed: "Min clearance: 0.2mm Min track: 0.2mm Min hole: 0.3mm Min annular ring: 0.15mm"

Commit message: wip pcb rev.A
Parts:
- added C42: 51p, PCM_Capacitor_THT_AKL:C_Disc_D5.0mm_W2.5mm_P2.50mm, F.Cu at (109.1, 176.7)
- added C43: 100n, PCM_Capacitor_THT_AKL:C_Disc_D5.0mm_W2.5mm_P2.50mm, F.Cu at (105.1, 208.8)
- added C44: 1u, PCM_Capacitor_THT_AKL:CP_Radial_D4.0mm_P2.00mm, F.Cu at (105.6, 205.4)
- added C45: 100n, PCM_Capacitor_THT_AKL:C_Disc_D5.0mm_W2.5mm_P2.50mm, F.Cu at (73.9, 175.4)
- added G***: LOGO, LOGO, F.Cu at (93.4, 170.2)
- added G***: LOGO, LOGO, F.Cu at (120.0, 171.1)
- added JP3: SolderJumper_2_Bridged, Jumper:SolderJumper-2_P1.3mm_Bridged_RoundedPad1.0x1.5mm, B.Cu at (114.7, 122.7)
- added R38: 10k, PCM_Resistor_THT_AKL:R_Axial_DIN0207_L6.3mm_D2.5mm_P7.62mm_Horizontal, F.Cu at (110.4, 214.8)
- added R39: 10k, PCM_Resistor_THT_AKL:R_Axial_DIN0207_L6.3mm_D2.5mm_P7.62mm_Horizontal, F.Cu at (110.4, 211.8)
- C12: value 2.2n -> 220p
- C13, C7: value 30p -> 18p
- C18: value 30p -> 330p
- C19: value 330p -> 30p
- C26: value 150p -> 100n
- C27: value 33u -> 10u
- C5: value 10u -> 4.7u
- L1: value 68uH/2A -> 47uH/2A
- Q1, Q2, Q3, Q4: value BC549B -> BC549
- RN1, RN2: footprint Resistor_THT:R_Array_SIP9 -> Resistor_THT:R_Array_SIP8
- U10: value MC1458P -> 4558D
- moved R9 17.3 mm to (94.2, 201.5)
- moved R5 10.4 mm to (102.8, 217.8), turned to 0 degrees
- moved C10 4.19 mm to (108.1, 208.8), turned to 0 degrees
- moved D4 2.34 mm to (105.3, 222.6)
- moved C12 1.83 mm to (71.4, 161.3)
- moved Q2 1.83 mm to (75.2, 171.1)
- moved R10 1.83 mm to (68.8, 164.4)
- moved R13 1.83 mm to (68.8, 167.5)
- moved C28 0.22 mm to (83.9, 201.5)
- moved U7 0.22 mm to (81.4, 211.8)
- moved R11 0.06 mm to (102.2, 196.6)
- moved R7 0.06 mm to (102.2, 187.6)
- moved R12 0.06 mm to (94.6, 193.6)
- moved R8 0.06 mm to (94.6, 190.6)
Connections:
- C10 pad 2: /SND_I -> Net-(JP3-B)
- J6 pad 2: /SND_I -> Net-(J6-Pad2)
- JP1 pad 2: /PPUCLK -> Net-(JP1-C)
- R10 pad 1: Net-(Q2-E) -> GND
- R14 pad 1: +5VA_2 -> Net-(Q4-B)
- R14 pad 2: Net-(Q4-B) -> +5VA_2
- R15 pad 1: Net-(Q4-B) -> GND
- R15 pad 2: GND -> Net-(Q4-B)
- R9 pad 1: Net-(U7-I6) -> Net-(JP3-B)
- R9 pad 2: /SND_I -> Net-(U7-I6)
- U7 pad 10: GND -> Net-(U7-I4)
- U7 pad 13: /SND_I -> Net-(JP3-B)
Routing:
- net /SND_I: track 201.8 -> 16.2 mm, vias 2 -> 0
- net Net-(JP3-B): track 0.00 -> 184.6 mm, vias 0 -> 3
- net +5V: track 810.8 -> 851.9 mm
- net /PPUCLK: track 37.4 -> 4.87 mm, vias 2 -> 0
- net Net-(JP1-C): track 0.00 -> 31.4 mm, vias 0 -> 2
- net Net-(U7-I4): track 0.00 -> 15.1 mm
- net Net-(J6-Pad2): track 0.00 -> 13.9 mm
- net +5VA_2: track 40.4 -> 53.9 mm
- net Net-(C44-Pad2): track 0.00 -> 9.10 mm
- net /~{RESET}: track 243.4 -> 235.5 mm, vias 3 -> 2
- net /A13: track 68.4 -> 74.5 mm
- net Net-(D4-K): track 11.7 -> 5.79 mm
- net /A14: track 70.2 -> 75.9 mm
- net /A12: track 61.0 -> 64.7 mm
- net /~{RAMSEL}: track 64.9 -> 61.4 mm, vias 1 -> 2
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Other:
- board text added: "${TITLE}"
- board text added: "+9-12V Any polarity"
- board text added: "21 MHz"
- board text added: "26 MHz"
- board text added: "CPU"
- board text added: "Eugene Lozovoy 2023 Rev.${REVISION}"
- board text added: "PPU"
- board text added: "SRAM"
