File: pcb/rev.A/dendy.kicad_sch (KiCad schematic)
At the start: 125 parts, among them J10 FC 60 pin cartridge slot, J2 DB15_Male, J3 RCJ-014, J4 RCJ-014, J5 PJ-322, J6 DB15_Male, J7 DS-210, J8 Conn_01x02, Q1 BC549B, Q2 BC549B, Q3 BC549B, Q4 BC549B, Q5 2N5401, SW1 SW_SPDT, SW2 Button THT, U1 74LS139, U10 MC1458P, U2 74LS373, U3 62256, U4 62256, U5 RP2A03, U6 RP2C02, U7 74LS368, U8 74LS368, U9 LM2596T-ADJ, Y1 21.47727MHz, Y2 26.601712MHz

Commit message: wip pcb rev.A
Parts:
- removed J5: PJ-322, my:PJ-322, symbol Connector:AudioJack4
- removed JP3: Jumper_2_Open, Connector_PinHeader_2.54mm:PinHeader_1x02_P2.54mm_Vertical, symbol Jumper:Jumper_2_Open
- added C36: 100u, PCM_Capacitor_THT_AKL:CP_Radial_D6.3mm_P2.50mm, symbol Device:C_Polarized
- added C37: 100n, PCM_Capacitor_THT_AKL:C_Disc_D5.0mm_W2.5mm_P2.50mm, symbol Device:C
- added J1: RCJ-014, my:CUI_RCJ-01X, symbol Connector:Conn_Coaxial
- added L4: 220u/0.2A, PCM_Inductor_THT_AKL:L_Radial_D8.7mm_P5.00mm_Fastron_07HCP, symbol Device:L
- added R44: 47k, PCM_Resistor_THT_AKL:R_Axial_DIN0207_L6.3mm_D2.5mm_P7.62mm_Horizontal, symbol Device:R
- added R45: 10k, PCM_Resistor_THT_AKL:R_Axial_DIN0207_L6.3mm_D2.5mm_P7.62mm_Horizontal, symbol Device:R
- C1, C10, C12, C13, C14, C15, C17, C18, C19, C20, C21, C26, C28, C29, C3, C30, C31, C32, C33, C34, C35, C7, C8, C9: footprint Capacitor_THT_AKL:C_Disc_D5.0mm_W2.5mm_P2.50mm -> PCM_Capacitor_THT_AKL:C_Disc_D5.0mm_W2.5mm_P2.50mm
- C11, C6: footprint Capacitor_THT_AKL:C_Trimmer_GKU_L5.6mm_W5.0mm_P5.8mm -> PCM_Capacitor_THT_AKL:C_Trimmer_GKU_L5.6mm_W5.0mm_P5.8mm
- C16: value 220u -> 100u; footprint Capacitor_THT_AKL:CP_Radial_D6.3mm_P2.50mm -> PCM_Capacitor_THT_AKL:CP_Radial_D6.3mm_P2.50mm; symbol Device:CP -> Device:C_Polarized
- C2: footprint Capacitor_THT_AKL:CP_Radial_D10.0mm_P5.00mm -> PCM_Capacitor_THT_AKL:CP_Radial_D10.0mm_P5.00mm; symbol Device:CP -> Device:C_Polarized
- C22, C23, C24, C25, C27, C5: footprint Capacitor_THT_AKL:CP_Radial_D4.0mm_P2.00mm -> PCM_Capacitor_THT_AKL:CP_Radial_D4.0mm_P2.00mm; symbol Device:CP -> Device:C_Polarized
- C4: footprint Capacitor_THT_AKL:CP_Radial_D8.0mm_P3.50mm -> PCM_Capacitor_THT_AKL:CP_Radial_D8.0mm_P3.50mm; symbol Device:CP -> Device:C_Polarized
- D2: footprint Diode_THT_AKL:D_DO-41_SOD81_P10.16mm_Horizontal -> PCM_Diode_THT_AKL:D_DO-41_SOD81_P10.16mm_Horizontal
- D3: footprint Diode_THT_AKL:D_DO-201AD_P15.24mm_Horizontal -> PCM_Diode_THT_AKL:D_DO-201AD_P15.24mm_Horizontal
- F1: value 0.5A -> 1A
- HOLE1, HOLE2, HOLE3, HOLE4, HOLE5, HOLE6, HOLE7: symbol Universal-ITX-Backplane-rescue:MountingHole_Pad-Mechanical-Universal-ITX-Backplane-rescue-Universal-ITX-Backplane-rescue -> Mechanical:MountingHole_Pad
- L1: footprint Inductor_SMD_AKL:L_12x12mm_H8mm -> PCM_Inductor_SMD_AKL:L_12x12mm_H8mm
- L2, L3: footprint Inductor_THT_AKL:L_Radial_D8.7mm_P5.00mm_Fastron_07HCP -> PCM_Inductor_THT_AKL:L_Radial_D8.7mm_P5.00mm_Fastron_07HCP
- Q1, Q2, Q3, Q4: footprint Package_TO_SOT_THT_AKL:TO-92_Inline_Wide_CBE -> PCM_Package_TO_SOT_THT_AKL:TO-92_Inline_Wide_CBE; symbol Transistor_BJT_AKL:BC549B -> PCM_Transistor_BJT_AKL:BC549B
- Q5: footprint Package_TO_SOT_THT_AKL:TO-92_Inline_Wide_EBC -> PCM_Package_TO_SOT_THT_AKL:TO-92_Inline_Wide_EBC; symbol Transistor_BJT_AKL:2N5401 -> PCM_Transistor_BJT_AKL:2N5401
- R1: value 100 -> 47k; footprint Resistor_THT_AKL:R_Axial_DIN0207_L6.3mm_D2.5mm_P7.62mm_Horizontal -> PCM_Resistor_THT_AKL:R_Axial_DIN0207_L6.3mm_D2.5mm_P7.62mm_Horizontal
- R10, R11, R12, R13, R14, R15, R16, R17, R18, R19, R2, R20, R21, R22, R23, R24, R25, R26, R27, R28, R29, R3, R30, R31, R32, R33, R34, R35, R36, R37, R38, R39, R4, R40, R41, R42, R43, R5, R6, R7, R8, R9: footprint Resistor_THT_AKL:R_Axial_DIN0207_L6.3mm_D2.5mm_P7.62mm_Horizontal -> PCM_Resistor_THT_AKL:R_Axial_DIN0207_L6.3mm_D2.5mm_P7.62mm_Horizontal
- RN2, RN3: value R_Network05 -> 10k; footprint Resistor_THT_AKL:R_Array_SIP6 -> PCM_Resistor_THT_AKL:R_Array_SIP6
- U1, U7, U8: footprint Package_DIP_AKL:DIP-16_W7.62mm -> PCM_Package_DIP_AKL:DIP-16_W7.62mm
- U10: footprint Package_DIP_AKL:DIP-8_W7.62mm_LongPads -> PCM_Package_DIP_AKL:DIP-8_W7.62mm_LongPads; symbol Amplifier_Operational_AKL:MC1458P -> PCM_Amplifier_Operational_AKL:MC1458P
- U2: footprint Package_DIP_AKL:DIP-20_W7.62mm -> PCM_Package_DIP_AKL:DIP-20_W7.62mm
- U3, U4: footprint Package_DIP_AKL:DIP-28_W7.62mm -> PCM_Package_DIP_AKL:DIP-28_W7.62mm
- U5, U6: footprint Package_DIP_AKL:DIP-40_W15.24mm_Socket -> PCM_Package_DIP_AKL:DIP-40_W15.24mm_Socket
- Y1, Y2: footprint Crystal_AKL:Crystal_HC49-U_Vertical -> PCM_Crystal_AKL:Crystal_HC49-U_Vertical
Connections:
- net +5V: now also L4.1
- net A0: now also U3.10 (A0); no longer U3.3 (A7)
- net A1: now also U3.9 (A1); no longer U3.4 (A6)
- net A10: now also U3.25 (A8); no longer U3.21 (A10)
- net A13: now also U1.14 (A0); no longer U1.2 (A0)
- net A14: now also U1.13 (A1); no longer U1.3 (A1)
- net A15: now also U1.3 (A1); no longer U1.13 (A1)
- net A2: now also U3.8 (A2); no longer U3.5 (A5)
- net A3: now also U3.21 (A10); no longer U3.6 (A4)
- net A5: now also U3.6 (A4); no longer U3.8 (A2)
- net A6: now also U3.5 (A5); no longer U3.9 (A1)
- net A7: now also U3.4 (A6); no longer U3.10 (A0)
- net A8: now also U3.24 (A9); no longer U3.25 (A8)
- net A9: now also U3.3 (A7); no longer U3.24 (A9)
- net COMPOSITE: now also J1.1 (In); no longer J4.1 (In)
- net D0: now also U3.15 (Q3); no longer U3.11 (Q0)
- net D1: now also U3.16 (Q4); no longer U3.12 (Q1)
- net D3: now also U3.17 (Q5); no longer U3.19 (Q7)
- net D4: now also U3.12 (Q1); no longer U3.18 (Q6)
- net D5: now also U3.18 (Q6); no longer U3.17 (Q5)
- net D6: now also U3.11 (Q0); no longer U3.16 (Q4)
- net D7: now also U3.19 (Q7); no longer U3.15 (Q3)
- net GND: now also R1.2, SW1.3 (C), U1.1 (E), C36.2, C37.1, J1.2 (Ext), R44.2; no longer U1.15 (E), U9.5 (~{ON}/OFF)
- net M2: now also U1.2 (A0); no longer U1.14 (A0)
- net PA0: now also U4.10 (A0); no longer U4.4 (A6)
- net PA1: now also U4.9 (A1); no longer U4.5 (A5)
- net PA3: now also U4.7 (A3); no longer U4.9 (A1)
- net PA4: now also U4.21 (A10); no longer U4.3 (A7)
- net PA5: now also U4.4 (A6); no longer U4.6 (A4)
- net PA6: now also U4.3 (A7); no longer U4.7 (A3)
- net PA7: now also U4.24 (A9); no longer U4.10 (A0)
- net PA8: now also U4.5 (A5); no longer U4.25 (A8)
- net PA9: now also U4.6 (A4); no longer U4.24 (A9)
- net PAD3: now also U4.15 (Q3); no longer U4.19 (Q7)
- net PAD4: now also U4.16 (Q4); no longer U4.18 (Q6)
- net PAD6: now also U4.18 (Q6); no longer U4.16 (Q4)
- net PAD7: now also U4.19 (Q7); no longer U4.15 (Q3)
- net SND_L: now also R44.1
- net SND_R: now also J4.1 (In), R1.1
- net VA10: now also U4.25 (A8); no longer U4.21 (A10)
- net ~{PPUSEL}: now also U1.11 (O1); no longer U1.5 (O1)
- net ~{ROMSEL}: now also U1.7 (O3); no longer U1.9 (O3)
- net at SW1.2 (B): now also U9.5 (~{ON}/OFF), R45.1; no longer F1.2
- net at D1.4: now also J7.2, J7.3; no longer SW1.3 (C)
- net at D5.2 (A), R4.2: now also U1.12 (O0); no longer U1.4 (O0)
- net at C24.1, R28.1: no longer R1.2
- net at C2.1, C3.1, D1.3 (+)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: now also R45.2
- net +5VA renamed +5VA_1
- net +5VA_1: no longer Q4.1 (C), R14.1
- new net: U1.15 (E), U1.5 (O1)
- new net: D1.2, F1.2
- new net +5VA_2: C36.1, C37.2, L4.2, Q4.1 (C), R14.1
Other:
- note added: "AUDIO OUTPUT"
- note added: "CLOCK"
- note added: "JOYSTICKS"
- note added: "POWER"
- note added: "VIDEO OUTPUT"
- moved on the sheet: C1, C10, C11, C12, C13, C14, C15, C16, C17, C2, C21, C23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

Commit message: wip pcb rev.A
Parts:
- removed J8: Conn_01x02, Connector_Molex:Molex_KK-254_AE-6410-02A_1x02_P2.54mm_Vertical, symbol Connector_Generic:Conn_01x02
- removed R38, R39, R40, R42: 10k, PCM_Resistor_THT_AKL:R_Axial_DIN0207_L6.3mm_D2.5mm_P7.62mm_Horizontal, symbol Device:R
- removed RN2, RN3: 10k, PCM_Resistor_THT_AKL:R_Array_SIP6, symbol Device:R_Network05
- added C38, C39, C40, C41: 100u, PCM_Capacitor_THT_AKL:CP_Radial_D6.3mm_P2.50mm, symbol Device:C_Polarized
- added D4: LED, LED_THT:LED_D5.0mm, symbol Device:LED
- added RN1, RN2: 10k, Resistor_THT:R_Array_SIP9, symbol Device:R_Network08
- L2: value 68uH/2A -> 47uH/2A
Connections:
- net +5V: now also C38.1, C39.1, C40.1, C41.1, D4.2 (A), RN1.1 (common), RN2.1 (common)
- net D0: now also U3.13 (Q2); no longer U3.15 (Q3)
- net D1: now also U3.15 (Q3); no longer U3.16 (Q4)
- net D2: now also U3.12 (Q1); no longer U3.13 (Q2)
- net D3: now also U3.16 (Q4); no longer U3.17 (Q5)
- net D4: now also U3.11 (Q0); no longer U3.12 (Q1)
- net D5: now also U3.17 (Q5); no longer U3.18 (Q6)
- net D6: now also U3.18 (Q6); no longer U3.11 (Q0)
- net GND: now also C38.2, C39.2, C40.2, C41.2
- net OUT0: now also RN1.5 (R4)
- net OUT1: now also RN1.7 (R6)
- net OUT2: now also RN1.8 (R7)
- net PA5: now also U4.5 (A5); no longer U4.4 (A6)
- net PA6: now also U4.25 (A8); no longer U4.3 (A7)
- net PA7: now also U4.4 (A6); no longer U4.24 (A9)
- net PA8: now also U4.24 (A9); no longer U4.5 (A5)
- net PAD0: now also U4.19 (Q7); no longer U4.11 (Q0)
- net PAD1: now also U4.18 (Q6); no longer U4.12 (Q1)
- net PAD2: now also U4.17 (Q5); no longer U4.13 (Q2)
- net PAD3: now also U4.16 (Q4); no longer U4.15 (Q3)
- net PAD4: now also U4.15 (Q3); no longer U4.16 (Q4)
- net PAD5: now also U4.13 (Q2); no longer U4.17 (Q5)
- net PAD6: now also U4.12 (Q1); no longer U4.18 (Q6)
- net PAD7: now also U4.11 (Q0); no longer U4.19 (Q7)
- net VA10: now also U4.3 (A7); no longer U4.25 (A8)
- net ~{IRQ}: now also RN2.7 (R6)
- net at R5.1: now also D4.1 (K)
- net at J6.13 (P13), U7.4 (I2): now also RN1.4 (R3)
- net at J2.9 (P9), J6.14 (P14), U7.7 (O3a): now also RN1.6 (R5)
- net at J6.4, U8.10 (I4): now also RN2.6 (R5)
- net at J6.5, U8.6 (I3): now also RN2.5 (R4)
- net at J6.6, U8.12 (I5): now also RN2.4 (R3)
- net at J6.7, U8.4 (I2): now also RN2.3 (R2)
- net at J6.8, U8.14 (I6): now also RN2.2 (R1)
- net at J6.9 (P9), U8.3 (O1a): now also RN2.8 (R7)
- net at J2.8, U7.2 (I1): now also RN1.2 (R1)
- no-connect marks 16 -> 18
Other:
- moved on the sheet: C1, C10, C28, C29, C30, C31, C32, C33, C34, C35, C4, C5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

Commit message: wip pcb rev.A
Parts:
- added C42: 51p, PCM_Capacitor_THT_AKL:C_Disc_D5.0mm_W2.5mm_P2.50mm, symbol Device:C
- added C43, C45: 100n, PCM_Capacitor_THT_AKL:C_Disc_D5.0mm_W2.5mm_P2.50mm, symbol Device:C
- added C44: 1u, PCM_Capacitor_THT_AKL:CP_Radial_D4.0mm_P2.00mm, symbol Device:C_Polarized
- added JP3: SolderJumper_2_Bridged, Jumper:SolderJumper-2_P1.3mm_Bridged_RoundedPad1.0x1.5mm, symbol Jumper:SolderJumper_2_Bridged
- added R38, R39: 10k, PCM_Resistor_THT_AKL:R_Axial_DIN0207_L6.3mm_D2.5mm_P7.62mm_Horizontal, symbol Device:R
- C12: value 2.2n -> 220p
- C13, C7: value 30p -> 18p
- C18: value 30p -> 330p
- C19: value 330p -> 30p
- C26: value 150p -> 100n
- C27: value 33u -> 10u
- C5: value 10u -> 4.7u
- L1: value 68uH/2A -> 47uH/2A; now left out of the parts list
- Q1, Q2, Q3, Q4: value BC549B -> BC549
- RN1, RN2: footprint Resistor_THT:R_Array_SIP9 -> Resistor_THT:R_Array_SIP8; symbol Device:R_Network08 -> Device:R_Network07
- U10: value MC1458P -> 4558D
- U3, U4: Label RAM -> SRAM
Connections:
- net +5V: now also C45.2
- net +5VA_2: now also R14.2; no longer R14.1
- net GND: now also R10.1, R15.1, C43.1, C45.1; no longer R15.2, U7.10 (I4)
- net PPUCLK: now also C42.2; no longer JP1.2 (C)
- net SND_I: now also JP3.1 (A); no longer C10.2, J6.2, R9.2, U7.13 (O6b)
- net at C12.1, Q2.3 (E), R13.1: no longer R10.1
- net at Q4.2 (B), Q5.1 (E): now also R14.1, R15.2; no longer R14.2, R15.1
- net at R9.1: now also C10.2, U7.13 (O6b), JP3.2 (B); no longer U7.14 (I6)
- new net: J6.2, R38.1, R39.1
- new net: C43.2, R38.2, U7.10 (I4)
- new net: C42.1, JP1.2 (C)
- new net: C44.1, R9.2, U7.14 (I6)
- new net: C44.2, R39.2
- no-connect marks 18 -> 16
Other:
- note added: "CPU"
- note added: "PPU"
- note added: "UA6527P HA6257P TA-03NP1 8Z01N MG-P-501"
- note added: "UA6538 HA6538 TA-02NP 8Z02 MG-P-502"
- title: (none) -> Dendy
- moved on the sheet: C12, C28, C29, C30, C31, C32, C33, C34, C35, Q2, R10, R13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

Commit message: wip pcb rev.A
Parts:
- added HOLE6: HOLE, MountingHole:MountingHole_3.2mm_M3_Pad_Via, symbol Mechanical:MountingHole_Pad
- C36: renamed from C6; symbol Device:CTRIM -> Device:C_Trim
- C37: renamed from C11; symbol Device:CTRIM -> Device:C_Trim
- J6: renamed from J2; Desc Joystick 1 -> Joypad 1
- J7: renamed from J6; Desc Joystick 2 -> Joypad 2
- SW2: renamed from SW1; footprint my:SS12F44G5 -> my:FC_Power_Switch_Universal
- renumbered C24 to C1, C25 to C10, C1 to C11, C16 to C12, C31 to C13, C33 to C14, C34 to C15, C32 to C16, C20 to C17, C30 to C18, C35 to C19, C41 to C20, C40 to C21, C18 to C22, C19 to C23, C12 to C24, C37 to C25, C21 to C26, C42 to C27, C45 to C28, C39 to C29, C26 to C3, C38 to C30, C36 to C31, C9 to C32, C7 to C33, C8 to C34, C5 to C35, C28 to C38, C29 to C39, C22 to C4, C15 to C40, C13 to C41, C14 to C42, C44 to C43, C43 to C44, C10 to C45, C23 to C5, C27 to C6, C17 to C7, C3 to C8, C4 to C9, D3 to D2, D2 to D3, D5 to D4, D4 to D5, HOLE5 to HOLE1, HOLE3 to HOLE2, HOLE6 to HOLE3, HOLE7 to HOLE5, HOLE2 to HOLE7, HOLE1 to HOLE8, J4 to J2, J7 to J4, J10 to J5, JP2 to JP1, JP1 to JP2, Q4 to Q1, Q5 to Q3, Q1 to Q4, Q3 to Q5, R20 to R1, R33 to R10, R2 to R11, R19 to R12, R3 to R13, R45 to R14, R23 to R15, R27 to R16, R21 to R17, R29 to R18, R35 to R19, R28 to R2, R18 to R20, R26 to R21, R34 to R22, R22 to R23, R30 to R24, R36 to R25, R31 to R26, R43 to R27, R4 to R28, R41 to R29, R1 to R3, R16 to R30, R10 to R31, R13 to R32, R14 to R33, R15 to R34, R7 to R35, R8 to R36, R12 to R37, R11 to R38, R6 to R39, R44 to R4, R9 to R40, R39 to R41, R38 to R42, R5 to R43, R24 to R5, R25 to R6, R37 to R7, R17 to R8, R32 to R9, SW2 to SW1, U9 to U1, U8 to U10, U10 to U2, U2 to U7, U1 to U8, U7 to U9
Connections:
- net GND: now also SW2.1 (A), HOLE6.1; no longer SW2.3 (C)
- net J1D1: now reaches J7.13 (P13), RN1.4 (R3), U9.4 (I2)
- net J1CLK: now reaches J6.9 (P9), J7.14 (P14), RN1.6 (R5), U9.7 (O3a)
- net J2MIC: now reaches J7.2, R41.1, R42.1
- net J2D4: now reaches J7.4, RN2.6 (R5), U10.10 (I4)
- net J2D3: now reaches J7.5, RN2.5 (R4), U10.6 (I3)
- net J2D2: now reaches J7.6, RN2.4 (R3), U10.12 (I5)
- net J2D1: now reaches J7.7, RN2.3 (R2), U10.4 (I2)
- net J2D0: now reaches J7.8, RN2.2 (R1), U10.14 (I6)
- net J2CLK: now reaches J7.9 (P9), RN2.8 (R7), U10.3 (O1a)
- net J1D0: now reaches J6.8, RN1.2 (R1), U9.2 (I1)
- net ~{JOY1} renamed ~{OE1}
- net ~{JOY2} renamed ~{OE2}
Other:
- note added: "For LM2596-5.0: R11 - 0 Ohm R13,C11 - do not install"
- note removed: "For LM2596-5.0: R1 - 0 Ohm R2,C1 - do not install"
- moved on the sheet: HOLE1, HOLE3, HOLE7, HOLE8, RN1, RN2, SW2

Commit message: pcb rev.A final version
Parts:
- added J6: Conn_01x05, Connector_Molex:Molex_KK-254_AE-6410-05A_1x05_P2.54mm_Vertical, symbol Connector_Generic:Conn_01x05
- added J7: Conn_01x06, Connector_Molex:Molex_KK-254_AE-6410-06A_1x06_P2.54mm_Vertical, symbol Connector_Generic:Conn_01x06
- J8: renamed from J6; symbol Connector:DB15_Male -> Connector:DA15_Plug; Desc Joypad 1 -> (none); Label (none) -> Joypad 1
- J9: renamed from J7; symbol Connector:DB15_Male -> Connector:DA15_Plug; Desc Joypad 2 -> (none); Label (none) -> Joypad 2
- L1: now in the parts list
- L2: now left out of the parts list
- R13: value 1k -> 976
- U10, U9: value 74LS368 -> 74HC368
- U3, U4: value 62256 -> 61C256; ValueAlt (none) -> 6264, 62128, 62256, AS7C256
- U5: value RP2A03 -> UA6527P; ValueAlt (none) -> HA6527P, TA-03NP, MG-P-501
- U6: value RP2C02 -> UA6538; ValueAlt (none) -> HA6538, TA-02NP, MG-P-502
- renumbered C3 to C2, C4 to C3, C2 to C4
Connections:
- net +5V: now also J6.5 (Pin_5), J7.6 (Pin_6); no longer U3.1 (A14), U3.2 (A12), U3.23 (A11), U4.1 (A14), U4.2 (A12), U4.23 (A11)
- net A0: now also U3.21 (A10); no longer U3.10 (A0)
- net A1: now also U3.10 (A0); no longer U3.9 (A1)
- net A2: now also U3.9 (A1); no longer U3.8 (A2)
- net A3: now also U3.8 (A2); no longer U3.21 (A10)
- net D1: now also U3.12 (Q1); no longer U3.15 (Q3)
- net D2: now also U3.11 (Q0); no longer U3.12 (Q1)
- net D3: now also U3.15 (Q3); no longer U3.16 (Q4)
- net D4: now also U3.16 (Q4); no longer U3.11 (Q0)
- net GND: now also U3.1 (A14), U3.2 (A12), U3.23 (A11), U4.1 (A14), U4.2 (A12), U4.23 (A11), J6.1 (Pin_1), J7.2 (Pin_2)
- net J1CLK: now also J6.4 (Pin_4)
- net J1D0: now also J6.2 (Pin_2)
- net J2CLK: now also J7.5 (Pin_5)
- net J2D0: now also J7.3 (Pin_3)
- net J2MIC: now also J7.1 (Pin_1)
- net OUT0: now also J6.3 (Pin_3), J7.4 (Pin_4)
Other:
- note removed: "CPU"
- note removed: "PPU"
- note removed: "UA6527P HA6257P TA-03NP1 8Z01N MG-P-501"
- note removed: "UA6538 HA6538 TA-02NP 8Z02 MG-P-502"
- moved on the sheet: C4, C8, D1, F1, J1, J2, Q1, Q3, R30, R33, R34, R4
